File: kicad/PicoM10_bld.kicad_pcb (KiCad board)
At the start: 6 copper layers, 8 x 10 mm, 20 parts, among them J1 Conn_Coaxial, U1 MIA-M10Q, U2 NCP160xMX

Commit message: test
Parts:
- moved D1 1.02 mm to (102.7, 102.2)
Routing:
- net Net-(D1-A): track 7.14 -> 4.77 mm
Changed lines of the file:
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@@
 		(sheetname "Root")
 		(sheetfile "PicoM10_bld.kicad_sch")
+		(clearance 0.2)
 		(fp_text user "${REFERENCE}"
 			(at 0 2.5 0)
@@
 		(sheetname "Root")
 		(sheetfile "PicoM10_bld.kicad_sch")
+		(clearance 0.2)
 		(fp_text user "${REFERENCE}"
 			(at 0 2.5 0)
@@
 		(sheetname "Root")
 		(sheetfile "PicoM10_bld.kicad_sch")
+		(clearance 0.2)
 		(fp_text user "${REFERENCE}"
 			(at 0 2.5 0)
@@
 		(sheetname "Root")
 		(sheetfile "PicoM10_bld.kicad_sch")
+		(clearance 0.2)
 		(fp_text user "${REFERENCE}"
 			(at 0 2.5 0)
@@
 	(footprint "Diode_SMD:D_SOD-923"
 		(layer "B.Cu")
-		(at 102.75 103.25 90)
+		(at 102.65 102.23 90)
 		(descr "https://www.onsemi.com/pub/Collateral/ESD9B-D.PDF#page=4")
 		(tags "Diode SOD923")
@@
 		(height 2.75)
 		(orientation 0)
-		(gr_text "8.00 mm"
+		(gr_text "8,00 mm"
 			(at 104 111.6 0)
 			(layer "Dwgs.User")
@@
 		(height 3.2)
 		(orientation 1)
-		(gr_text "10.00 mm"
+		(gr_text "10,00 mm"
 			(at 109.85 105 90)
 			(layer "Dwgs.User")
@@
 	)
 	(segment
-		(start 103.55 102.87)
-		(end 103.65 102.87)
-		(width 0.25)
-		(layer "B.Cu")
-		(net 2)
-	)
-	(segment
 		(start 104.36 103.675)
 		(end 104.36 103.025)
@@
 	)
 	(segment
-		(start 102.75 103.67)
-		(end 103.55 102.87)
+		(start 102.65 102.65)
+		(end 102.87 102.87)
+		(width 0.25)
+		(layer "B.Cu")
+		(net 2)
+	)
+	(segment
+		(start 102.87 102.87)
+		(end 103.65 102.87)
 		(width 0.25)
 		(layer "B.Cu")
@@
 	)
 	(segment
+		(start 102.65 101.81)
+		(end 101.44 101.81)
+		(width 0.25)
+		(layer "F.Cu")
+		(net 4)
+	)
+	(segment
 		(start 101.07 101.18)
 		(end 101 101.25)
@@
 		(net 4)
 	)
+	(segment
+		(start 101.44 101.81)
+		(end 101.25 102)
+		(width 0.25)
+		(layer "F.Cu")
+		(net 4)
+	)
 	(via
-		(at 101.25 102)
+		(at 101.25 100.5)
 		(size 0.45)
 		(drill 0.2)
@@
 	)
 	(via
-		(at 101.25 100.65)
+		(at 102.65 101.81)
 		(size 0.45)
 		(drill 0.2)
@@
 	)
 	(via
-		(at 102.75 102.85)
+		(at 101.25 102)
 		(size 0.45)
 		(drill 0.2)
@@
 		(end 101.25 100.65)
 		(width 0.25)
-		(layer "In2.Cu")
-		(net 4)
-	)
-	(segment
-		(start 101.9 102)
-		(end 101.25 102)
-		(width 0.25)
-		(layer "In2.Cu")
-		(net 4)
-	)
-	(segment
-		(start 102.75 102.85)
-		(end 101.9 102)
-		(width 0.25)
-		(layer "In2.Cu")
-		(net 4)
-	)
-	(segment
-		(start 101.9 102)
-		(end 101.9 101.3)
-		(width 0.25)
-		(layer "In2.Cu")
+		(layer "B.Cu")
 		(net 4)
 	)
 	(segment
-		(start 101.9 101.3)
-		(end 101.25 100.65)
+		(start 100.82 101.18)
+		(end 100.75 101.25)
 		(width 0.25)
-		(layer "In3.Cu")
+		(layer "B.Cu")
 		(net 4)
 	)
 	(segment
-		(start 102.75 102.85)
-		(end 101.9 102)
+		(start 102.09 101.81)
+		(end 102.65 101.81)
 		(width 0.25)
-		(layer "In3.Cu")
+		(layer "B.Cu")
 		(net 4)
 	)
@@
 		(end 101.25 102)
 		(width 0.25)
-		(layer "In3.Cu")
+		(layer "B.Cu")
 		(net 4)
 	)
@@
 		(end 101.9 101.3)
 		(width 0.25)
-		(layer "In3.Cu")
+		(layer "B.Cu")
 		(net 4)
 	)
 	(segment
-		(start 100.82 101.18)
-		(end 100.75 101.25)
+		(start 101.9 102)
+		(end 102.09 101.81)
 		(width 0.25)
 		(layer "B.Cu")
@@
 		(net 1)
 		(net_name "GND")
-		(layer "F.Cu")
+		(layers "F&B.Cu")
 		(hatch edge 0.5)
 		(priority 2)
@@
 			(pts
 				(xy 102.5 100) (xy 102.5 102.25) (xy 102 102.75) (xy 100 102.75) (xy 100 104.75) (xy 102 104.75)
-				(xy 102.5 105.25) (xy 102.5 110) (xy 107.75 110) (xy 107.75 100)
+				(xy 102.5 105.25) (xy 102.5 110) (xy 108 110) (xy 108 100)
 			)
 		)
@@
 		(polygon
 			(pts
-				(xy 101.75 104.75) (xy 100 104.75) (xy 100 102.75) (xy 101.75 102.75) (xy 101.75 100) (xy 107.75 100)
-				(xy 107.75 110) (xy 101.75 110)
+				(xy 100 105) (xy 100 105) (xy 100 102.5) (xy 100 102.5) (xy 100 100) (xy 108 100) (xy 108 110) (xy 100 110)
 			)
 		)
@@
 		(layers "In2.Cu" "In3.Cu")
 		(hatch edge 0.5)
-		(priority 1)
 		(connect_pads yes
 			(clearance 0.1)
@@
 		(polygon
 			(pts
-				(xy 101.75 100) (xy 107.75 100) (xy 107.75 110) (xy 101.75 110)
+				(xy 100 105) (xy 100 102.5) (xy 100 100) (xy 108 100) (xy 108 110) (xy 100 110)
 			)
 		)
 	)
 	(zone
-		(net 1)
-		(net_name "GND")
+		(net 0)
+		(net_name "")
 		(layer "B.Cu")
 		(hatch edge 0.5)
-		(priority 3)
 		(connect_pads yes
-			(clearance 0.1)
+			(clearance 0)
 		)
 		(min_thickness 0.1)
 		(filled_areas_thickness no)
-		(fill yes
+		(keepout
+			(tracks allowed)
+			(vias allowed)
+			(pads allowed)
+			(copperpour not_allowed)
+			(footprints allowed)
+		)
+		(fill
 			(thermal_gap 0.5)
 			(thermal_bridge_width 0.5)
@@
 		(polygon
 			(pts
-				(xy 102.5 100) (xy 102.5 102.25) (xy 102 102.75) (xy 100 102.75) (xy 100 104.75) (xy 102 104.75)
-				(xy 102.5 105.25) (xy 102.5 110) (xy 107.75 110) (xy 107.75 100)
+				(xy 103.55 105.7) (xy 105.75 105.7) (xy 105.75 107.7) (xy 103.55 107.7)
 			)
 		)

Commit message: minor schematic and layout updates
Routing:
- net GNSS_Rx: track 7.94 -> 4.77 mm
- net Net-(R1-Pad1): track 6.63 -> 4.18 mm
- net Net-(D1-A): track 4.77 -> 3.81 mm
- net GND: vias 18 -> 21
